Commit message: add: 导航(nano_demo测试良好)

File: src/dr100/dr100/urdf/dr100_controller.xacro (robot description, xacro)
@@ -47,4 +47,25 @@
             <robotBaseFrame>base_link</robotBaseFrame>
         </plugin>
+    </gazebo>
+    <!-- IMU -->
+    <gazebo reference="imu_base">
+        <material>Gazebo/Bule</material>
+        <gravity>true</gravity>
+        <sensor name="imu_sensor" type="imu">
+            <always_on>true</always_on>
+            <update_rate>100</update_rate>
+            <visualize>true</visualize>
+            <topic>__default_topic__</topic>
+            <plugin filename="libgazebo_ros_imu_sensor.so" name="imu_plugin">
+                <topicName>imu/data</topicName>
+                <bodyName>imu_base</bodyName>
+                <updateRateHZ>100.0</updateRateHZ>
+                <gaussianNoise>0.01</gaussianNoise>
+                <xyzOffset>0 0 0</xyzOffset>
+                <rpyOffset>0 0 0</rpyOffset>
+                <frameName>imu_base</frameName>
+            </plugin>
+            <pose>0 0 0 0 0 0</pose>
+        </sensor>
     </gazebo>
     <!-- Gazebo requires the robosense_gazebo_plugins package -->

File: src/dr100/dr100/urdf/dr100_imu.xacro (robot description, xacro)
@@ -32,25 +32,4 @@
             <xacro:Box_inertial_matrix m = "${imu_mass}" l = "${imu_size}" w = "${imu_size}" h = "${imu_size}"/>
         </link>
-        <!-- Referenced link -->
-        <gazebo reference="imu_base">
-            <material>Gazebo/Bule</material>
-            <gravity>true</gravity>
-            <sensor name="imu_sensor" type="imu">
-                <always_on>true</always_on>
-                <update_rate>100</update_rate>
-                <visualize>true</visualize>
-                <topic>__default_topic__</topic>
-                <plugin filename="libgazebo_ros_imu_sensor.so" name="imu_plugin">
-                    <topicName>imu/data</topicName>
-                    <bodyName>imu_base</bodyName>
-                    <updateRateHZ>100.0</updateRateHZ>
-                    <gaussianNoise>0.01</gaussianNoise>
-                    <xyzOffset>0 0 0</xyzOffset>
-                    <rpyOffset>0 0 0</rpyOffset>
-                    <frameName>imu_base</frameName>
-                </plugin>
-                <pose>0 0 0 0 0 0</pose>
-            </sensor>
-        </gazebo>
     </xacro:macro>
 </robot>
