Commit message: add: 添加仿真驱动

File: src/dr100/dr100/urdf/dr100.xacro (robot description, xacro)
@@ -31,5 +31,5 @@
             <mass value="40" />
             <origin xyz="0.0 0.0 0.0" />
-            <inertia ixx="3.791" ixy="-0.012" ixz="0.007" iyy="7.879" iyz="-141.459" izz="9.703" />
+            <inertia ixx="3.791" ixy="-0.012" ixz="0.007" iyy="7.879" iyz="0.023" izz="9.703" />
         </inertial>
     </link>

File: src/dr100/dr100/urdf/dr100_controller.xacro (robot description, xacro)
@@ -1,5 +1,5 @@
 <?xml version="1.0"?>
 <robot name="dr100_controller" xmlns:xacro="http://wiki.ros.org/xacro">
-    <xacro:arg name="gpu" default="false"/>
+    <xacro:arg name="gpu" default="true"/>
     <xacro:property name="gpu" value="$(arg gpu)" />
     <xacro:property name="M_PI" value="3.14159"/>

Commit message: 实机调试

File: src/dr100/dr100/urdf/dr100.xacro (robot description, xacro)
@@ -52,10 +52,10 @@
     <xacro:include filename="$(find dr100)/urdf/dr100_imu.xacro" />
     <xacro:imu sensor_name="imu" parent_link="base_link">
-        <origin xyz="0.25 0 0.5355" rpy="0 0 0"/>
+        <origin xyz="0.265 0 0.5355" rpy="0 0 0"/>
     </xacro:imu>
     <!-- LiDAR -->
     <xacro:include filename="$(find dr100)/urdf/dr100_lidar.xacro"/>
     <xacro:robosense name="robosense" parent_link="base_link">
-        <origin xyz="0.2500 0 0.5725" rpy="0 0 0" />
+        <origin xyz="0.265 0 0.5725" rpy="0 0 0" />
     </xacro:robosense>
 </robot>
